Commit message: update aubo i7 new urdf model and moveit config

File: aubo_description/urdf/aubo_i7.urdf (robot description, URDF)
Before this commit: robot aubo_i7, 8 links, 7 joints
Links:
- added link pedestal_Link; visual box size=1.0 1.0 0.1
- link base_link: mass 1.23448927826401 -> 0.76802; geometry collision mesh filename=package://aubo_description/meshes/aubo_i7/collision/base_li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; visual mesh filename=package://aubo_description/meshes/aubo_i7/collision/base_li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
- link foreArm_Link: mass 2.88724337413486 -> 2.1062; geometry collision mesh filename=package://aubo_description/meshes/aubo_i7/collision/foreArm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; visual mesh filename=package://aubo_description/meshes/aubo_i7/collision/foreArm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
- link shoulder_Link: mass 9.88740003439705 -> 1.8535; geometry collision mesh filename=package://aubo_description/meshes/aubo_i7/collision/shoulde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; visual mesh filename=package://aubo_description/meshes/aubo_i7/collision/shoulde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
- link upperArm_Link: mass 4.46934833776782 -> 5.4; geometry collision mesh filename=package://aubo_description/meshes/aubo_i7/collision/upperAr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; visual mesh filename=package://aubo_description/meshes/aubo_i7/collision/upperAr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
- link wrist1_Link: mass 0.579814564711146 -> 0.59073; geometry collision mesh filename=package://aubo_description/meshes/aubo_i7/collision/wrist1_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; visual mesh filename=package://aubo_description/meshes/aubo_i7/collision/wrist1_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
- link wrist2_Link: mass 0.579814565182749 -> 0.59073; geometry collision mesh filename=package://aubo_description/meshes/aubo_i7/collision/wrist2_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; visual mesh filename=package://aubo_description/meshes/aubo_i7/collision/wrist2_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
- link wrist3_Link: mass 0.136689987013058 -> 0.13549; geometry collision mesh filename=package://aubo_description/meshes/aubo_i7/collision/wrist3_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; visual mesh filename=package://aubo_description/meshes/aubo_i7/collision/wrist3_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
Joints:
- removed joint foreArm_Joint
- removed joint shoulder_Joint
- removed joint upperArm_Joint
- removed joint wrist1_Joint
- removed joint wrist2_Joint
- removed joint wrist3_Joint
- added joint foreArm_joint: type revolute, parent upperArm_Link, child foreArm_Link, origin xyz=0.368 0 0 rpy=-3.1416 0 0, axis 0 0 1, limit lower=-3.05 upper=3.05 effort=300 velocity=100
- added joint pedestal_joint: type fixed, parent pedestal_Link, child base_link, origin xyz=0 0 0.051 rpy=0 0 0
- added joint shoulder_joint: type revolute, parent base_link, child shoulder_Link, origin xyz=0 0 0.122 rpy=0 0 3.1416, axis 0 0 1, limit lower=-3.05 upper=3.05 effort=133 velocity=2.5964
- added joint upperArm_joint: type revolute, parent shoulder_Link, child upperArm_Link, origin xyz=0 0.1215 0 rpy=-1.5708 -1.5708 0, axis 0 0 1, limit lower=-3.05 upper=3.05 effort=133 velocity=2.5964
- added joint wrist1_joint: type revolute, parent foreArm_Link, child wrist1_Link, origin xyz=0.316 0 0 rpy=3.1416 0 1.5708, axis 0 0 1, limit lower=-3.05 upper=3.05 effort=300 velocity=100
- added joint wrist2_joint: type revolute, parent wrist1_Link, child wrist2_Link, origin xyz=0 0.1025 0 rpy=-1.5708 0 0, axis 0 0 1, limit lower=-3.05 upper=3.05 effort=300 velocity=100
- added joint wrist3_joint: type revolute, parent wrist2_Link, child wrist3_Link, origin xyz=0 -0.094 0 rpy=1.5708 0 0, axis 0 0 1, limit lower=-3.05 upper=3.05 effort=300 velocity=100
- joint world_joint: child base_link -> pedestal_Link; origin xyz=0.0 0.0 0.0 rpy=0.0 0.0 0.0 -> xyz=0 0 0.05 rpy=0 0 0
